File: hardware/sonpakharu.kicad_sch (KiCad schematic)
At the start: 58 parts, among them IC1 ESP32-S3-WROOM-1U-N4, J10 EXT2, J11 EXT3, J12 BATT, J13 EXT7, J14 PWR, J15 EXT8, J16 485, J17 ESP PRG, J3 ADC2, J4 ADC1, J5 EXT4, J6 I2C, J7 EXT5, J8 EXT1, J9 EXT6, Q1 DMG3415U, Q4 S8050, SW1 ON/OFF, U1 AP2112K-3.3TRG1, U2 MCP73831-2-OT, U3 MCP3426Axx-xSN, U4 MAX485E

Commit message: added IO4 pin to connector
Parts:
- removed J11: EXT3, Connector_Molex:Molex_KK-254_AE-6410-02A_1x02_P2.54mm_Vertical, symbol Connector_Generic:Conn_01x02
- added J1: EXT3, Connector_Molex:Molex_KK-254_AE-6410-03A_1x03_P2.54mm_Vertical, symbol Connector_Generic:Conn_01x03
Connections:
- net IO19: now also J1.2 (Pin_2)
- net IO20: now also J1.1 (Pin_1)
- net IO4: now also J1.3 (Pin_3)
Changed lines of the file:
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@@
 	(wire
 		(pts
-			(xy 252.73 80.01) (xy 255.27 80.01)
-		)
-		(stroke
-			(width 0)
-			(type default)
-		)
-	)
-	(wire
-		(pts
 			(xy 137.16 82.55) (xy 139.7 82.55)
 		)
@@
 	(wire
 		(pts
+			(xy 252.73 82.55) (xy 255.27 82.55)
+		)
+		(stroke
+			(width 0)
+			(type default)
+		)
+	)
+	(wire
+		(pts
 			(xy 78.74 44.45) (xy 78.74 55.88)
 		)
@@
 	(wire
 		(pts
+			(xy 252.73 77.47) (xy 255.27 77.47)
+		)
+		(stroke
+			(width 0)
+			(type default)
+		)
+	)
+	(wire
+		(pts
 			(xy 163.83 29.21) (xy 163.83 35.56)
 		)
@@
 	(wire
 		(pts
-			(xy 247.65 153.67) (xy 247.65 156.21)
+			(xy 252.73 80.01) (xy 255.27 80.01)
 		)
 		(stroke
@@
 	(wire
 		(pts
-			(xy 224.79 138.43) (xy 222.25 138.43)
+			(xy 247.65 153.67) (xy 247.65 156.21)
 		)
 		(stroke
@@
 	(wire
 		(pts
-			(xy 109.22 160.02) (xy 105.41 160.02)
+			(xy 224.79 138.43) (xy 222.25 138.43)
 		)
 		(stroke
@@
 	(wire
 		(pts
-			(xy 137.16 74.93) (xy 139.7 74.93)
+			(xy 109.22 160.02) (xy 105.41 160.02)
 		)
 		(stroke
@@
 	(wire
 		(pts
-			(xy 252.73 82.55) (xy 255.27 82.55)
+			(xy 137.16 74.93) (xy 139.7 74.93)
 		)
 		(stroke
@@
 		)
 	)
+	(label "IO19"
+		(at 255.27 80.01 0)
+		(fields_autoplaced yes)
+		(effects
+			(font
+				(size 1.27 1.27)
+			)
+			(justify left bottom)
+		)
+	)
 	(label "IO39"
 		(at 210.82 93.98 0)
@@
 		)
 	)
+	(label "IO4"
+		(at 255.27 77.47 0)
+		(fields_autoplaced yes)
+		(effects
+			(font
+				(size 1.27 1.27)
+			)
+			(justify left bottom)
+		)
+	)
 	(label "RX"
 		(at 196.85 135.89 0)
@@
 		)
 	)
-	(label "IO4"
-		(at 165.1 147.32 0)
-		(fields_autoplaced yes)
-		(effects
-			(font
-				(size 1.27 1.27)
-			)
-			(justify left bottom)
-		)
-	)
 	(label "IO37"
 		(at 210.82 83.82 0)
@@
 		)
 	)
-	(label "IO19"
-		(at 255.27 80.01 0)
-		(fields_autoplaced yes)
-		(effects
-			(font
-				(size 1.27 1.27)
-			)
-			(justify left bottom)
-		)
-	)
 	(label "D+"
 		(at 266.7 140.97 0)
@@
 	)
 	(label "IO0"
-		(at 69.85 116.84 0)
+		(at 67.31 116.84 0)
 		(fields_autoplaced yes)
 		(effects
@@
 	)
 	(symbol
+		(lib_id "Connector_Generic:Conn_01x03")
+		(at 247.65 80.01 180)
+		(unit 1)
+		(exclude_from_sim no)
+		(in_bom yes)
+		(on_board yes)
+		(dnp no)
+		(property "Reference" "J1"
+			(at 247.65 74.93 0)
+			(effects
+				(font
+					(size 1.27 1.27)
+				)
+			)
+		)
+		(property "Value" "EXT3"
+			(at 243.84 80.01 90)
+			(effects
+				(font
+					(size 1.27 1.27)
+				)
+			)
+		)
+		(property "Footprint" "Connector_Molex:Molex_KK-254_AE-6410-03A_1x03_P2.54mm_Vertical"
+			(at 247.65 80.01 0)
+			(effects
+				(font
+					(size 1.27 1.27)
+				)
+				(hide yes)
+			)
+		)
+		(property "Datasheet" "~"
+			(at 247.65 80.01 0)
+			(effects
+				(font
+					(size 1.27 1.27)
+				)
+				(hide yes)
+			)
+		)
+		(property "Description" ""
+			(at 247.65 80.01 0)
+			(effects
+				(font
+					(size 1.27 1.27)
+				)
+				(hide yes)
+			)
+		)
+		(pin "1"
+		)
+		(pin "2"
+		)
+		(pin "3"
+		)
+		(instances
+			(project "sonpakharu"
+				(path "/7446772e-77ef-4971-88a7-8e2cc94b8894"
+					(reference "J1")
+					(unit 1)
+				)
+			)
+		)
+	)
+	(symbol
 		(lib_id "Mechanical:MountingHole_Pad")
 		(at 140.97 189.23 0)
@@
 					(unit 1)
 				)
-			)
-		)
-	)
-	(symbol
-		(lib_id "Connector_Generic:Conn_01x02")
-		(at 247.65 82.55 180)
-		(unit 1)
-		(exclude_from_sim no)
-		(in_bom yes)
-		(on_board yes)
-		(dnp no)
-		(property "Reference" "J11"
-			(at 247.65 77.47 0)
-			(effects
-				(font
-					(size 1.27 1.27)
-				)
-			)
-		)
-		(property "Value" "EXT3"
-			(at 243.84 81.28 90)
-			(effects
-				(font
-					(size 1.27 1.27)
-				)
-			)
-		)
-		(property "Footprint" "Connector_Molex:Molex_KK-254_AE-6410-02A_1x02_P2.54mm_Vertical"
-			(at 247.65 82.55 0)
-			(effects
-				(font
-					(size 1.27 1.27)
-				)
-				(hide yes)
-			)
-		)
-		(property "Datasheet" "~"
-			(at 247.65 82.55 0)
-			(effects
-				(font
-					(size 1.27 1.27)
-				)
-				(hide yes)
-			)
-		)
-		(property "Description" ""
-			(at 247.65 82.55 0)
-			(effects
-				(font
-					(size 1.27 1.27)
-				)
-				(hide yes)
-			)
-		)
-		(pin "1"
-		)
-		(pin "2"
-		)
-		(instances
-			(project "sonpakharu"
-				(path "/7446772e-77ef-4971-88a7-8e2cc94b8894"
-					(reference "J11")
-					(unit 1)
-				)

Commit message: Fix: layout u[dated
Parts:
- IC1: footprint KiCad:ESP32S3WROOM1UN4 -> ESP32S3WROOM1UN4
- Q4: footprint Package_TO_SOT_SMD:SOT-23 -> Package_TO_SOT_THT:TO-92_Inline
- U1: footprint AP2112K_3_3TRG1:SOT25 -> SOT_RG1_DIO
